File: connectors.kicad_sch (KiCad schematic)
At the start: 22 parts, among them J2 Barrel Jack, J3 15P JST, P1 2P JST, P2 2P JST, P3 2P JST, P4 2P JST

Commit message: Finalized V2
Parts:
- C10, C11, C12, C13, C14, C9: footprint Capacitor_SMD:C_0402_1005Metric -> Capacitor_SMD:C_0402_1005Metric_Pad0.74x0.62mm_HandSolder
- D7: footprint Diode_SMD:D_0402_1005Metric -> Diode_SMD:D_0402_1005Metric_Pad0.77x0.64mm_HandSolder
- R11: renamed from R8; footprint Resistor_SMD:R_0402_1005Metric -> Resistor_SMD:R_0402_1005Metric_Pad0.72x0.64mm_HandSolder
- R12: renamed from R9; footprint Resistor_SMD:R_0402_1005Metric -> Resistor_SMD:R_0402_1005Metric_Pad0.72x0.64mm_HandSolder
- R13: renamed from R10; footprint Resistor_SMD:R_0402_1005Metric -> Resistor_SMD:R_0402_1005Metric_Pad0.72x0.64mm_HandSolder
- R14: renamed from R11; footprint Resistor_SMD:R_0402_1005Metric -> Resistor_SMD:R_0402_1005Metric_Pad0.72x0.64mm_HandSolder
- R15: renamed from R12; footprint Resistor_SMD:R_0402_1005Metric -> Resistor_SMD:R_0402_1005Metric_Pad0.72x0.64mm_HandSolder
- R16: renamed from R13; footprint Resistor_SMD:R_0402_1005Metric -> Resistor_SMD:R_0402_1005Metric_Pad0.72x0.64mm_HandSolder
Other:
- note added: "CAN"
- note removed: "CANBUS"
