File: bms.kicad_pcb (KiCad board)
At the start: 2 copper layers, 92 x 59.2 mm, 204 parts, among them IC1 RAA489204, J1 USB_C_Receptacle_USB2.0_14P, P3 2P JST, Q1 NPN, Q2 SiRA00DP, Q3 SiRA00DP, Q4 SiRA00DP, Q5 SiRA00DP, U1 LMR36510ADDA, U2 ESP32-C6-MINI-1, U3 SN65HVD230, U4 BQ25756RRVR, U5 TPS25730D, U6 MAX17614ATP+, U7 MAX17614ATP+

Commit message: Finalized V2
Parts:
- removed the JP1 at (110.5, 80.2)
- added +USBV: TEST POINT, TestPoint:TestPoint_Pad_1.0x1.0mm, F.Cu at (134.1, 92.3)
- added +VBAT: TEST POINT, TestPoint:TestPoint_Pad_1.0x1.0mm, F.Cu at (149.4, 55.0)
- added +VBUCK: TEST POINT, TestPoint:TestPoint_Pad_1.0x1.0mm, F.Cu at (165.1, 49.2)
- added +VPLUG: TEST POINT, TestPoint:TestPoint_Pad_1.0x1.0mm, F.Cu at (113.5, 83.7)
- added 1: TEST POINT, TestPoint:TestPoint_Pad_1.0x1.0mm, F.Cu at (165.9, 80.2)
- added 10: TEST POINT, TestPoint:TestPoint_Pad_1.0x1.0mm, F.Cu at (136.9, 67.3)
- added 11: TEST POINT, TestPoint:TestPoint_Pad_1.0x1.0mm, F.Cu at (136.9, 63.7)
- added 12: TEST POINT, TestPoint:TestPoint_Pad_1.0x1.0mm, F.Cu at (136.9, 61.2)
- added 13: TEST POINT, TestPoint:TestPoint_Pad_1.0x1.0mm, F.Cu at (136.9, 58.9)
- added 14: TEST POINT, TestPoint:TestPoint_Pad_1.0x1.0mm, F.Cu at (177.1, 47.5)
- added 2: TEST POINT, TestPoint:TestPoint_Pad_1.0x1.0mm, F.Cu at (163.4, 80.2)
- added 3: TEST POINT, TestPoint:TestPoint_Pad_1.0x1.0mm, F.Cu at (161.0, 80.2)
- added 4: TEST POINT, TestPoint:TestPoint_Pad_1.0x1.0mm, F.Cu at (158.6, 80.2)
- added 5: TEST POINT, TestPoint:TestPoint_Pad_1.0x1.0mm, F.Cu at (156.2, 80.2)
- added 6: TEST POINT, TestPoint:TestPoint_Pad_1.0x1.0mm, F.Cu at (153.8, 80.2)
- added 7: TEST POINT, TestPoint:TestPoint_Pad_1.0x1.0mm, F.Cu at (151.4, 80.2)
- added 8: TEST POINT, TestPoint:TestPoint_Pad_1.0x1.0mm, F.Cu at (149.0, 80.2)
- added 9: TEST POINT, TestPoint:TestPoint_Pad_1.0x1.0mm, F.Cu at (136.9, 69.8)
- added GND: TEST POINT, TestPoint:TestPoint_Pad_1.0x1.0mm, F.Cu at (177.1, 72.5)
- added H1: MountingHole, MountingHole:MountingHole_3.2mm_M3, F.Cu at (88.0, 37.0)
- added H2: MountingHole, MountingHole:MountingHole_3.2mm_M3, F.Cu at (184.0, 37.0)
- added H3: MountingHole, MountingHole:MountingHole_3.2mm_M3, F.Cu at (88.0, 101.0)
- added H4: MountingHole, MountingHole:MountingHole_3.2mm_M3, F.Cu at (184.0, 101.0)
- added PPHV: TEST POINT, TestPoint:TestPoint_Pad_1.0x1.0mm, F.Cu at (126.1, 79.1)
- added R10: 10k, Resistor_SMD:R_0402_1005Metric_Pad0.72x0.64mm_HandSolder, F.Cu at (131.5, 91.4)
- added R8: 120, Resistor_SMD:R_0402_1005Metric_Pad0.72x0.64mm_HandSolder, F.Cu at (106.9, 81.4)
- added R9: 0, Resistor_SMD:R_0402_1005Metric_Pad0.72x0.64mm_HandSolder, F.Cu at (104.7, 81.4)
- added U3: TLV70433DBVR, Package_TO_SOT_SMD:SOT-23-5_HandSoldering, F.Cu at (127.9, 87.0)
- added U5: LM66200DRLR, Package_TO_SOT_SMD:SOT-23-8, F.Cu at (132.1, 88.9)
- C1, C10, C11, C12, C13, C14, C15, C16, C17, C18, C19, C2, C20, C21, C22, C23, C24, C25, C26, C27, C28, C29, C3, C30, C31, C32, C33, C34, C35, C36, C37, C38, C39, C4, C40, C41, C42, C43, C44, C45, C46, C47, C48, C49, C5, C50, C51, C52, C53, C54, C55, C56, C57, C58, C59, C6, C60, C61, C62, C63, C64, C65, C66, C67, C68, C69, C7, C70, C71, C72, C73, C74, C75, C76, C77, C78, C79, C8, C9: footprint Capacitor_SMD:C_0402_1005Metric -> Capacitor_SMD:C_0402_1005Metric_Pad0.74x0.62mm_HandSolder
- D1, D10, D11, D2, D3, D4, D5, D6, D7, D8, D9: footprint Diode_SMD:D_0402_1005Metric -> Diode_SMD:D_0402_1005Metric_Pad0.77x0.64mm_HandSolder
- R1, R2, R3, R4, R5, R6, R7: footprint Resistor_SMD:R_0402_1005Metric -> Resistor_SMD:R_0402_1005Metric_Pad0.72x0.64mm_HandSolder
- R11: renamed from R8; footprint Resistor_SMD:R_0402_1005Metric -> Resistor_SMD:R_0402_1005Metric_Pad0.72x0.64mm_HandSolder
- R12: renamed from R9; footprint Resistor_SMD:R_0402_1005Metric -> Resistor_SMD:R_0402_1005Metric_Pad0.72x0.64mm_HandSolder
- R13: renamed from R10; footprint Resistor_SMD:R_0402_1005Metric -> Resistor_SMD:R_0402_1005Metric_Pad0.72x0.64mm_HandSolder
- R14: renamed from R11; footprint Resistor_SMD:R_0402_1005Metric -> Resistor_SMD:R_0402_1005Metric_Pad0.72x0.64mm_HandSolder
- R15: renamed from R12; footprint Resistor_SMD:R_0402_1005Metric -> Resistor_SMD:R_0402_1005Metric_Pad0.72x0.64mm_HandSolder
- R16: renamed from R13; footprint Resistor_SMD:R_0402_1005Metric -> Resistor_SMD:R_0402_1005Metric_Pad0.72x0.64mm_HandSolder
- R17: renamed from R14; footprint Resistor_SMD:R_0402_1005Metric -> Resistor_SMD:R_0402_1005Metric_Pad0.72x0.64mm_HandSolder
- R18: renamed from R15; footprint Resistor_SMD:R_0402_1005Metric -> Resistor_SMD:R_0402_1005Metric_Pad0.72x0.64mm_HandSolder
- R19: renamed from R16; footprint Resistor_SMD:R_0402_1005Metric -> Resistor_SMD:R_0402_1005Metric_Pad0.72x0.64mm_HandSolder
- R20: renamed from R17; footprint Resistor_SMD:R_0402_1005Metric -> Resistor_SMD:R_0402_1005Metric_Pad0.72x0.64mm_HandSolder
- R21: renamed from R18; footprint Resistor_SMD:R_0402_1005Metric -> Resistor_SMD:R_0402_1005Metric_Pad0.72x0.64mm_HandSolder
- R22: renamed from R19; footprint Resistor_SMD:R_0402_1005Metric -> Resistor_SMD:R_0402_1005Metric_Pad0.72x0.64mm_HandSolder
- R23: renamed from R20; footprint Resistor_SMD:R_0402_1005Metric -> Resistor_SMD:R_0402_1005Metric_Pad0.72x0.64mm_HandSolder
- R24: renamed from R21; footprint Resistor_SMD:R_0402_1005Metric -> Resistor_SMD:R_0402_1005Metric_Pad0.72x0.64mm_HandSolder
- R25: renamed from R22; footprint Resistor_SMD:R_0402_1005Metric -> Resistor_SMD:R_0402_1005Metric_Pad0.72x0.64mm_HandSolder
- R26: renamed from R23; footprint Resistor_SMD:R_0402_1005Metric -> Resistor_SMD:R_0402_1005Metric_Pad0.72x0.64mm_HandSolder
- R27: renamed from R24; footprint Resistor_SMD:R_0402_1005Metric -> Resistor_SMD:R_0402_1005Metric_Pad0.72x0.64mm_HandSolder
- R28: renamed from R25; footprint Resistor_SMD:R_0402_1005Metric -> Resistor_SMD:R_0402_1005Metric_Pad0.72x0.64mm_HandSolder
- R29: renamed from R26; footprint Resistor_SMD:R_0402_1005Metric -> Resistor_SMD:R_0402_1005Metric_Pad0.72x0.64mm_HandSolder
- R30: renamed from R27; footprint Resistor_SMD:R_0402_1005Metric -> Resistor_SMD:R_0402_1005Metric_Pad0.72x0.64mm_HandSolder
- R31: renamed from R28; footprint Resistor_SMD:R_0402_1005Metric -> Resistor_SMD:R_0402_1005Metric_Pad0.72x0.64mm_HandSolder
- R32: renamed from R29; footprint Resistor_SMD:R_0402_1005Metric -> Resistor_SMD:R_0402_1005Metric_Pad0.72x0.64mm_HandSolder
- R33: renamed from R30; footprint Resistor_SMD:R_0402_1005Metric -> Resistor_SMD:R_0402_1005Metric_Pad0.72x0.64mm_HandSolder
- R34: renamed from R31; footprint Resistor_SMD:R_0402_1005Metric -> Resistor_SMD:R_0402_1005Metric_Pad0.72x0.64mm_HandSolder
- R35: renamed from R32; footprint Resistor_SMD:R_0402_1005Metric -> Resistor_SMD:R_0402_1005Metric_Pad0.72x0.64mm_HandSolder
- R36: renamed from R33; footprint Resistor_SMD:R_0402_1005Metric -> Resistor_SMD:R_0402_1005Metric_Pad0.72x0.64mm_HandSolder
- R37: renamed from R34; footprint Resistor_SMD:R_0402_1005Metric -> Resistor_SMD:R_0402_1005Metric_Pad0.72x0.64mm_HandSolder
- R38: renamed from R35; footprint Resistor_SMD:R_0402_1005Metric -> Resistor_SMD:R_0402_1005Metric_Pad0.72x0.64mm_HandSolder
- R39: renamed from R36; footprint Resistor_SMD:R_0402_1005Metric -> Resistor_SMD:R_0402_1005Metric_Pad0.72x0.64mm_HandSolder
- R40: renamed from R37; footprint Resistor_SMD:R_0402_1005Metric -> Resistor_SMD:R_0402_1005Metric_Pad0.72x0.64mm_HandSolder
- R41: renamed from R38; footprint Resistor_SMD:R_0402_1005Metric -> Resistor_SMD:R_0402_1005Metric_Pad0.72x0.64mm_HandSolder
- R42: renamed from R39; footprint Resistor_SMD:R_0402_1005Metric -> Resistor_SMD:R_0402_1005Metric_Pad0.72x0.64mm_HandSolder
- R43: renamed from R40; footprint Resistor_SMD:R_0402_1005Metric -> Resistor_SMD:R_0402_1005Metric_Pad0.72x0.64mm_HandSolder
- R44: renamed from R41; footprint Resistor_SMD:R_0402_1005Metric -> Resistor_SMD:R_0402_1005Metric_Pad0.72x0.64mm_HandSolder
- R45: renamed from R42; footprint Resistor_SMD:R_0402_1005Metric -> Resistor_SMD:R_0402_1005Metric_Pad0.72x0.64mm_HandSolder
- R46: renamed from R43; footprint Resistor_SMD:R_0402_1005Metric -> Resistor_SMD:R_0402_1005Metric_Pad0.72x0.64mm_HandSolder
- R47: renamed from R44; footprint Resistor_SMD:R_0402_1005Metric -> Resistor_SMD:R_0402_1005Metric_Pad0.72x0.64mm_HandSolder
- R48: renamed from R45; footprint Resistor_SMD:R_0402_1005Metric -> Resistor_SMD:R_0402_1005Metric_Pad0.72x0.64mm_HandSolder
- R49: renamed from R47; footprint Resistor_SMD:R_0402_1005Metric -> Resistor_SMD:R_0402_1005Metric_Pad0.72x0.64mm_HandSolder
- R50: renamed from R48; footprint Resistor_SMD:R_0402_1005Metric -> Resistor_SMD:R_0402_1005Metric_Pad0.72x0.64mm_HandSolder
- R51: renamed from R49; footprint Resistor_SMD:R_0402_1005Metric -> Resistor_SMD:R_0402_1005Metric_Pad0.72x0.64mm_HandSolder
- R52: renamed from R50; footprint Resistor_SMD:R_0402_1005Metric -> Resistor_SMD:R_0402_1005Metric_Pad0.72x0.64mm_HandSolder
- R53: renamed from R51; footprint Resistor_SMD:R_0402_1005Metric -> Resistor_SMD:R_0402_1005Metric_Pad0.72x0.64mm_HandSolder
- R54: renamed from R52; footprint Resistor_SMD:R_0402_1005Metric -> Resistor_SMD:R_0402_1005Metric_Pad0.72x0.64mm_HandSolder
- R55: renamed from R53; footprint Resistor_SMD:R_0402_1005Metric -> Resistor_SMD:R_0402_1005Metric_Pad0.72x0.64mm_HandSolder
- R56: renamed from R54; footprint Resistor_SMD:R_0402_1005Metric -> Resistor_SMD:R_0402_1005Metric_Pad0.72x0.64mm_HandSolder
- R57: renamed from R55; footprint Resistor_SMD:R_0402_1005Metric -> Resistor_SMD:R_0402_1005Metric_Pad0.72x0.64mm_HandSolder
- R58: renamed from R56; footprint Resistor_SMD:R_0402_1005Metric -> Resistor_SMD:R_0402_1005Metric_Pad0.72x0.64mm_HandSolder
- R59: renamed from R57; footprint Resistor_SMD:R_0402_1005Metric -> Resistor_SMD:R_0402_1005Metric_Pad0.72x0.64mm_HandSolder
- R60: renamed from R58; footprint Resistor_SMD:R_0402_1005Metric -> Resistor_SMD:R_0402_1005Metric_Pad0.72x0.64mm_HandSolder
- R61: renamed from R59; footprint Resistor_SMD:R_0402_1005Metric -> Resistor_SMD:R_0402_1005Metric_Pad0.72x0.64mm_HandSolder
- R62: renamed from R60; footprint Resistor_SMD:R_0402_1005Metric -> Resistor_SMD:R_0402_1005Metric_Pad0.72x0.64mm_HandSolder
- R63: renamed from R61; footprint Resistor_SMD:R_0402_1005Metric -> Resistor_SMD:R_0402_1005Metric_Pad0.72x0.64mm_HandSolder
- R64: renamed from R62; footprint Resistor_SMD:R_0402_1005Metric -> Resistor_SMD:R_0402_1005Metric_Pad0.72x0.64mm_HandSolder
- R65: renamed from R63; footprint Resistor_SMD:R_0402_1005Metric -> Resistor_SMD:R_0402_1005Metric_Pad0.72x0.64mm_HandSolder
- R66: renamed from R64; footprint Resistor_SMD:R_0402_1005Metric -> Resistor_SMD:R_0402_1005Metric_Pad0.72x0.64mm_HandSolder
- R67: renamed from R65; footprint Resistor_SMD:R_0402_1005Metric -> Resistor_SMD:R_0402_1005Metric_Pad0.72x0.64mm_HandSolder
- R68: renamed from R66; footprint Resistor_SMD:R_0402_1005Metric -> Resistor_SMD:R_0402_1005Metric_Pad0.72x0.64mm_HandSolder
- R69: renamed from R67; footprint Resistor_SMD:R_0402_1005Metric -> Resistor_SMD:R_0402_1005Metric_Pad0.72x0.64mm_HandSolder
- R70: renamed from R68; footprint Resistor_SMD:R_0402_1005Metric -> Resistor_SMD:R_0402_1005Metric_Pad0.72x0.64mm_HandSolder
- R71: renamed from R69; footprint Resistor_SMD:R_0402_1005Metric -> Resistor_SMD:R_0402_1005Metric_Pad0.72x0.64mm_HandSolder
- R72: renamed from R70; footprint Resistor_SMD:R_0402_1005Metric -> Resistor_SMD:R_0402_1005Metric_Pad0.72x0.64mm_HandSolder
- R73: renamed from R71; footprint Resistor_SMD:R_0402_1005Metric -> Resistor_SMD:R_0402_1005Metric_Pad0.72x0.64mm_HandSolder
- R74: renamed from R72; footprint Resistor_SMD:R_0402_1005Metric -> Resistor_SMD:R_0402_1005Metric_Pad0.72x0.64mm_HandSolder
- R75: renamed from R73; footprint Resistor_SMD:R_0402_1005Metric -> Resistor_SMD:R_0402_1005Metric_Pad0.72x0.64mm_HandSolder
- R76: renamed from R74; footprint Resistor_SMD:R_0402_1005Metric -> Resistor_SMD:R_0402_1005Metric_Pad0.72x0.64mm_HandSolder
- R77: renamed from R75; footprint Resistor_SMD:R_0402_1005Metric -> Resistor_SMD:R_0402_1005Metric_Pad0.72x0.64mm_HandSolder
- R78: renamed from R76; footprint Resistor_SMD:R_0402_1005Metric -> Resistor_SMD:R_0402_1005Metric_Pad0.72x0.64mm_HandSolder
- R79: renamed from R77; footprint Resistor_SMD:R_0402_1005Metric -> Resistor_SMD:R_0402_1005Metric_Pad0.72x0.64mm_HandSolder
- R80: renamed from R78; footprint Resistor_SMD:R_0402_1005Metric -> Resistor_SMD:R_0402_1005Metric_Pad0.72x0.64mm_HandSolder
- R81: renamed from R79; footprint Resistor_SMD:R_0402_1005Metric -> Resistor_SMD:R_0402_1005Metric_Pad0.72x0.64mm_HandSolder
- R82: renamed from R80; footprint Resistor_SMD:R_0402_1005Metric -> Resistor_SMD:R_0402_1005Metric_Pad0.72x0.64mm_HandSolder
- R83: renamed from R81; footprint Resistor_SMD:R_0402_1005Metric -> Resistor_SMD:R_0402_1005Metric_Pad0.72x0.64mm_HandSolder
- R84: renamed from R82; footprint Resistor_SMD:R_0402_1005Metric -> Resistor_SMD:R_0402_1005Metric_Pad0.72x0.64mm_HandSolder
- R85: renamed from R83; footprint Resistor_SMD:R_0402_1005Metric -> Resistor_SMD:R_0402_1005Metric_Pad0.72x0.64mm_HandSolder
- R86: renamed from R84; footprint Resistor_SMD:R_0402_1005Metric -> Resistor_SMD:R_0402_1005Metric_Pad0.72x0.64mm_HandSolder
- R87: renamed from R85; footprint Resistor_SMD:R_0402_1005Metric -> Resistor_SMD:R_0402_1005Metric_Pad0.72x0.64mm_HandSolder
- R88: renamed from R86; footprint Resistor_SMD:R_0402_1005Metric -> Resistor_SMD:R_0402_1005Metric_Pad0.72x0.64mm_HandSolder
- R89: renamed from R87; footprint Resistor_SMD:R_0402_1005Metric -> Resistor_SMD:R_0402_1005Metric_Pad0.72x0.64mm_HandSolder
- moved R11 27.1 mm to (153.3, 86.5), turned to 180 degrees
- moved R12 23.3 mm to (162.2, 86.5), turned to 180 degrees
- moved R13 23.1 mm to (170.9, 86.5), turned to 180 degrees
- moved R7 5.19 mm to (109.1, 78.6)
- moved D5 3.80 mm to (103.6, 82.6), turned to 0 degrees
- moved D6 3.80 mm to (108.0, 82.6), turned to 180 degrees
- moved C2 3.03 mm to (169.5, 52.7)
- moved C3 3.03 mm to (170.6, 52.7)
- moved D1 3.03 mm to (168.4, 52.7)
- moved C8 2.60 mm to (162.8, 48.7)
- moved C7 2.60 mm to (169.2, 42.4)
- moved L1 2.60 mm to (164.9, 45.5)
- moved U1 2.60 mm to (170.5, 47.2)
- moved C5 2.57 mm to (171.1, 41.9)
- moved R5 2.57 mm to (172.3, 41.9)
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- renumbered JP2 to JP1, NTC to P2, VIN to PLUG, U3 to U4, U4 to U6, U5 to U7, U6 to U8, U7 to U9
Connections:
- C8 pad 1: +3.3V -> +VBUCK
- D5 pad 2: Net-(D5-A2) -> CANL
- D6 pad 2: Net-(D6-A2) -> CANH
- FL1 pad 1: Net-(D5-A2) -> CANH
- FL1 pad 2: Net-(D6-A2) -> CANL
- L1 pad 2: +3.3V -> +VBUCK
- R5 pad 1: +3.3V -> +VBUCK
- R7 pad 2: Net-(JP1-A) -> Net-(U4-Rs)
- U2 pad 10: DBG_ACC -> USBFAULT
- U2 pad 12: PLUGFLIP -> SINKEN
- U2 pad 13: USBFAULT -> PLUGEVENT
- U2 pad 15: DRAIN -> CANRX
- U2 pad 16: unconnected-(U2-IO7-Pad16) -> CANTX
- U2 pad 19: CANTX -> DRAIN
- U2 pad 20: CANRX -> unconnected-(U2-IO15-Pad20)
- U2 pad 5: PLUGEVENT -> CAP_MIS
- U2 pad 6: CAP_MIS -> DBG_ACC
- U2 pad 9: SINKEN -> PLUGFLIP
- U4 pad 6: Net-(D5-A2) -> CANL
- U4 pad 7: Net-(D6-A2) -> CANH
- U4 pad 8: Net-(JP1-C) -> Net-(U4-Rs)
Routing:
- net +VBAT: track 0.00 -> 145.8 mm, vias 0 -> 7
- net +3.3V: track 0.00 -> 116.7 mm, vias 0 -> 6
- net +VBUCK: track 0.00 -> 82.4 mm, vias 0 -> 2
- net /Charge IC/PPHV: track 0.00 -> 75.7 mm, vias 0 -> 5
- net GND: track 0.00 -> 65.0 mm, vias 0 -> 293
- net +USBV: track 0.00 -> 64.3 mm
- net /BMS Controller/TEMPREG: track 0.00 -> 49.3 mm, vias 0 -> 3
- net /BMS Controller/CONN11: track 0.00 -> 47.8 mm, vias 0 -> 4
- net CANRX: track 0.00 -> 47.4 mm
- net /BMS Controller/CONN9: track 0.00 -> 47.2 mm, vias 0 -> 3
- net /BMS Controller/CONN10: track 0.00 -> 46.7 mm, vias 0 -> 3
- net /BMS Controller/CONN12: track 0.00 -> 46.4 mm, vias 0 -> 4
- net /BMS Controller/CONN13: track 0.00 -> 46.0 mm, vias 0 -> 4
- net USB_D-: track 0.00 -> 45.9 mm
- net USB_D+: track 0.00 -> 45.8 mm
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- added copper zone on F.Cu, net +3.3V
- added copper zone on F.Cu, net +USBV
- added copper zone on F.Cu, net +VPLUG
- added copper zone on F.Cu, net /Charge IC/PPHV
- added copper zone on F.Cu, net /Charge IC/SW1
- added copper zone on F.Cu, net /Charge IC/SW2
- added copper zone on F.Cu, net CANH
- added copper zone on F.Cu, net CANL
- added copper zone on F.Cu, net DRAIN
- added copper zone on B.Cu, net GND
- added copper zone on F.Cu, net GND
- added copper zone on In1.Cu, net GND
- added copper zone on In2.Cu, net GND
- added copper zone on F.Cu, net Net-(U1-SW)
- added copper zone on F.Cu, net Net-(U8-IN-Pad1)
Other:
- board size 92 x 59.2 mm -> 106 x 74 mm
- copper layers 2 -> 4
- board text removed: "BMS V1"
- board text removed: "MATTHEW EMBAYE"

Commit message: Finalized design for review and order
Other:
- board text added: "MATTHEW EMBAYE"

Commit message: Fixed Ideal Diodes
Parts:
- renumbered PPHV to +PPHV, PLUG to J2, BATTERY to J3, CAN to P1, NTC to P4, RESET to SW1, FLASH to SW2, +USBV to TP1, 7 to TP10, 6 to TP11, 5 to TP12, 4 to TP13, 3 to TP14, 2 to TP15, 1 to TP16, GND to TP17, +VBAT to TP18, +VBUCK to TP2, +VPLUG to TP20, 14 to TP3, 13 to TP4, 12 to TP5, 11 to TP6, 10 to TP7, 9 to TP8, 8 to TP9
Connections:
- +PPHV pad 1: /Charge IC/PPHV -> +PPHV
- C66 pad 2: /Charge IC/PPHV -> +PPHV
- C67 pad 2: /Charge IC/PPHV -> +PPHV
- C68 pad 1: /Charge IC/PPHV -> /Charge IC/OROUT
- C71 pad 2: /Charge IC/PPHV -> +PPHV
- C73 pad 2: /Charge IC/PPHV -> /Charge IC/OROUT
- C75 pad 2: +USBV -> +PPHV
- C78 pad 2: /Charge IC/PPHV -> /Charge IC/OROUT
- C79 pad 2: /Charge IC/PPHV -> /Charge IC/OROUT
- D11 pad 2: +USBV -> +PPHV
- Q2 pad 3: /Charge IC/PPHV -> /Charge IC/OROUT
- R78 pad 1: +USBV -> +PPHV
- R82 pad 1: +USBV -> +PPHV
- U6 pad 32: /Charge IC/PPHV -> /Charge IC/OROUT
- U6 pad 33: /Charge IC/PPHV -> /Charge IC/OROUT
- U6 pad 34: /Charge IC/PPHV -> /Charge IC/OROUT
- U7 pad 20: /Charge IC/PPHV -> +PPHV
- U8 pad 13: /Charge IC/PPHV -> /Charge IC/OROUT
- U8 pad 14: /Charge IC/PPHV -> /Charge IC/OROUT
- U8 pad 15: /Charge IC/PPHV -> /Charge IC/OROUT
- U9 pad 1: +USBV -> +PPHV
- U9 pad 13: /Charge IC/PPHV -> /Charge IC/OROUT
- U9 pad 14: /Charge IC/PPHV -> /Charge IC/OROUT
- U9 pad 15: /Charge IC/PPHV -> /Charge IC/OROUT
- U9 pad 2: +USBV -> +PPHV
- U9 pad 3: +USBV -> +PPHV
Routing:
- net /Charge IC/PPHV: track 75.7 -> 0.00 mm, vias 5 -> 0
- net /Charge IC/OROUT: track 0.00 -> 67.6 mm, vias 0 -> 4
- net +PPHV: track 0.00 -> 19.7 mm, vias 0 -> 2
- net +USBV: track 64.3 -> 52.2 mm
- net Net-(R55-Pad2): track 0.00 -> 1.04 mm
- added copper zone on F.Cu, net +PPHV
- added copper zone on F.Cu, net /Charge IC/OROUT
- removed copper zone on F.Cu, net /Charge IC/PPHV
Other:
- board text added: "+PPHV"
- board text added: "+USBV"
- board text added: "+VBAT"
- board text added: "+VBUCK"
- board text added: "+VPLUG"
- board text added: "1"
- board text added: "10"
- board text added: "11"
- board text added: "12"
- board text added: "13"
- board text added: "14"
- board text added: "2"
- board text added: "3"
- board text added: "4"
- board text added: "5"
- board text added: "6"
- board text added: "7"
- board text added: "8"
- board text added: "9"
- board text added: "BATTERY"
- board text added: "BOOT"
- board text added: "CAN"
- board text added: "GND"
- board text added: "MAIN"
- board text added: "RESET"
- board text added: "TEMP"

Commit message: EM-BMS1
good to order!
Parts:
- added C80: 0.1uF, Capacitor_SMD:C_0402_1005Metric_Pad0.74x0.62mm_HandSolder, F.Cu at (127.3, 90.0)
- added C81: 1uF, Capacitor_SMD:C_0402_1005Metric_Pad0.74x0.62mm_HandSolder, F.Cu at (130.2, 89.2)
- added C84: 100nF, Capacitor_SMD:C_0402_1005Metric_Pad0.74x0.62mm_HandSolder, F.Cu at (106.5, 70.6)
- added C85: 22uF, Capacitor_SMD:C_0402_1005Metric_Pad0.74x0.62mm_HandSolder, F.Cu at (107.5, 70.6)
- C44: value idk -> 47nF
- C47: value idk -> 2.2uF
- C50, C63, C69, C70, C78, C79: value 4.7µF -> 4.7uF
- C52, C57, C66: value 10µF -> 10uF
- C67, C71: value 22µF -> 22uF
- C73, C76: value 80µF -> 80uF
- D2, D4: value 65V TVS -> 5V TVS
- L1: value 22µH -> 22uH
- U4: value SN65HVD230 -> SN65HVD232
- moved R8 1.30 mm to (106.9, 80.1)
- moved R9 1.30 mm to (104.7, 80.1)
- moved U5 0.70 mm to (132.8, 88.9)
- moved R10 0.70 mm to (132.2, 91.4)
- moved TP1 0.30 mm to (134.4, 92.3)
- renumbered +PPHV to TP19
Connections:
- U2 pad 6: DBG_ACC -> unconnected-(U2-IO3-Pad6)
- U7 pad 10: DBG_ACC -> unconnected-(U7-DBG_ACC-Pad10)
Routing:
- net DBG_ACC: track 38.2 -> 0.00 mm, vias 2 -> 0
- net GND: track 65.0 -> 70.5 mm, vias 293 -> 299
- net +3.3V: track 116.7 -> 117.8 mm
- net +VLDO: track 2.21 -> 2.99 mm
- net +VBUCK: track 82.4 -> 81.7 mm
