File: bms.kicad_sch (KiCad schematic)
At the start: 32 parts, among them J1 USB_C_Receptacle_USB2.0_14P, SW1 Button, SW2 Button, U1 LMR36510ADDA, U2 ESP32-C6-MINI-1, U3 SN65HVD230

Commit message: Finalized V2
Parts:
- removed TP2: TEST POINT, symbol Connector:TestPoint
- added H1, H2, H3, H4: MountingHole, MountingHole:MountingHole_3.2mm_M3, symbol Mechanical:MountingHole
- added R10: 10k, Resistor_SMD:R_0402_1005Metric_Pad0.72x0.64mm_HandSolder, symbol Device:R_Small_US
- added R8: 120, Resistor_SMD:R_0402_1005Metric_Pad0.72x0.64mm_HandSolder, symbol Device:R_Small_US
- added R9: 0, Resistor_SMD:R_0402_1005Metric_Pad0.72x0.64mm_HandSolder, symbol Device:R_Small_US
- added U3: TLV70433DBVR, Package_TO_SOT_SMD:SOT-23-5_HandSoldering, symbol components:TLV704
- added U5: LM66200DRLR, Package_TO_SOT_SMD:SOT-23-8, symbol components:LM66200
- C1, C2, C3, C4, C5, C6, C7, C8: footprint Capacitor_SMD:C_0402_1005Metric -> Capacitor_SMD:C_0402_1005Metric_Pad0.74x0.62mm_HandSolder
- D1, D2, D3, D4, D5, D6: footprint Diode_SMD:D_0402_1005Metric -> Diode_SMD:D_0402_1005Metric_Pad0.77x0.64mm_HandSolder
- R1, R2, R3, R4, R5, R6, R7: footprint Resistor_SMD:R_0402_1005Metric -> Resistor_SMD:R_0402_1005Metric_Pad0.72x0.64mm_HandSolder
- TP1: renamed from TP23; footprint (none) -> TestPoint:TestPoint_Pad_1.0x1.0mm
- TP2: renamed from TP1; footprint (none) -> TestPoint:TestPoint_Pad_1.0x1.0mm
- renumbered U3 to U4
Connections:
- net +3.3V: now also R10.2, U5.2 (VOUT1), U5.7 (VOUT2); no longer C8.1, L1.2, R5.1, TP2.1
- net +USBV: now also U3.2 (VIN)
- net CANH: now also D6.2 (A2), FL1.1, U4.7 (CANH), R8.2
- net CANL: now also D5.2 (A2), FL1.2, U4.6 (CANL), R9.1
- net CANRX: now also U2.15 (IO6); no longer U2.20 (IO15)
- net CANTX: now also U2.16 (IO7); no longer U2.19 (IO14)
- net CAP_MIS: now also U2.5 (IO2); no longer U2.6 (IO3)
- net DBG_ACC: now also U2.6 (IO3); no longer U2.10 (IO5)
- net DRAIN: now also U2.19 (IO14); no longer U2.15 (IO6)
- net GND: now also U3.1 (GND), U5.1 (GND), U5.4 (ON), U5.5 (GND)
- net PLUGEVENT: now also U2.13 (IO1); no longer U2.5 (IO2)
- net PLUGFLIP: now also U2.9 (IO4); no longer U2.12 (IO0)
- net SINKEN: now also U2.12 (IO0); no longer U2.9 (IO4)
- net USBFAULT: now also U2.10 (IO5); no longer U2.13 (IO1)
- new net: R8.1, R9.2
- new net: U3.4 (NC), U3.5 (NC)
- new net: R10.1, U5.8 (ST)
- new net +VBUCK: C8.1, L1.2, R5.1, TP2.1, U5.3 (VIN1)
- new net +VLDO: U3.3 (VOUT), U5.6 (VIN2)
Other:
- note added: "3V3 IDEAL DIODE OR"
- note added: "LDO"
- note added: "MH"
- note removed: "differential routing"

Commit message: EM-BMS1
good to order!
Parts:
- added C80: 0.1uF, Capacitor_SMD:C_0402_1005Metric_Pad0.74x0.62mm_HandSolder, symbol Device:C_Small
- added C81: 1uF, Capacitor_SMD:C_0402_1005Metric_Pad0.74x0.62mm_HandSolder, symbol Device:C_Small
- added C84: 100nF, Capacitor_SMD:C_0402_1005Metric_Pad0.74x0.62mm_HandSolder, symbol Device:C_Small
- added C85: 22uF, Capacitor_SMD:C_0402_1005Metric_Pad0.74x0.62mm_HandSolder, symbol Device:C_Small
- D2, D4: value 65V TVS -> 5V TVS
- L1: value 22µH -> 22uH
- U4: value SN65HVD230 -> SN65HVD232
Connections:
- net +3.3V: now also C84.1, C85.1
- net +USBV: now also C80.1
- net +VLDO: now also C81.1
- net GND: now also C80.2, C81.2, C84.2, C85.2
- net DBG_ACC: no longer names the net of U2.6 (IO3)
- no-connect marks 3 -> 4
Other:
- sheet Charge IC ports: added none; removed DBG_ACC
- moved on the sheet: D5, D6, FL1, H1, H2, H3, H4, R10, R7, R8, R9, U3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
